Commit message: Added hx5-d20 meshes
Signed-off-by: Hyunwoo Nam <nhw@robotis.com>

File: motion_controller_models/models/hx5_d20/hx5_d20_left.urdf (robot description, URDF)
Before this commit: robot hx5_d20_left, 26 links, 25 joints
Links:
- link finger_end_l_link1: geometry visual box size=0.01 0.01 0.01
- link finger_end_l_link2: geometry visual box size=0.01 0.01 0.01
- link finger_end_l_link3: geometry visual box size=0.01 0.01 0.01
- link finger_end_l_link4: geometry visual box size=0.01 0.01 0.01
- link finger_end_l_link5: geometry visual box size=0.01 0.01 0.01
- link finger_l_link1: geometry collision mesh filename=package://motion_controller_models/models/hx5_d20/meshes/hx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 scale=0.001 0.001 0.001; visual mesh filename=package://motion_controller_models/models/hx5_d20/meshes/hx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 scale=0.001 0.001 0.001
- link finger_l_link10: geometry collision mesh filename=package://motion_controller_models/models/hx5_d20/meshes/hx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 scale=0.001 0.001 0.001; visual mesh filename=package://motion_controller_models/models/hx5_d20/meshes/hx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 scale=0.001 0.001 0.001
- link finger_l_link11: geometry collision mesh filename=package://motion_controller_models/models/hx5_d20/meshes/hx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 scale=0.001 0.001 0.001; visual mesh filename=package://motion_controller_models/models/hx5_d20/meshes/hx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 scale=0.001 0.001 0.001
- link finger_l_link12: geometry collision mesh filename=package://motion_controller_models/models/hx5_d20/meshes/hx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 scale=0.001 0.001 0.001; visual mesh filename=package://motion_controller_models/models/hx5_d20/meshes/hx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 scale=0.001 0.001 0.001
- link finger_l_link13: geometry collision mesh filename=package://motion_controller_models/models/hx5_d20/meshes/hx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 scale=0.001 0.001 0.001; visual mesh filename=package://motion_controller_models/models/hx5_d20/meshes/hx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 scale=0.001 0.001 0.001
- link finger_l_link14: geometry collision mesh filename=package://motion_controller_models/models/hx5_d20/meshes/hx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 scale=0.001 0.001 0.001; visual mesh filename=package://motion_controller_models/models/hx5_d20/meshes/hx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 scale=0.001 0.001 0.001
- link finger_l_link15: geometry collision mesh filename=package://motion_controller_models/models/hx5_d20/meshes/hx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 scale=0.001 0.001 0.001; visual mesh filename=package://motion_controller_models/models/hx5_d20/meshes/hx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 scale=0.001 0.001 0.001
- link finger_l_link16: geometry collision mesh filename=package://motion_controller_models/models/hx5_d20/meshes/hx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 scale=0.001 0.001 0.001; visual mesh filename=package://motion_controller_models/models/hx5_d20/meshes/hx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 scale=0.001 0.001 0.001
- link finger_l_link17: geometry collision mesh filename=package://motion_controller_models/models/hx5_d20/meshes/hx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 scale=0.001 0.001 0.001; visual mesh filename=package://motion_controller_models/models/hx5_d20/meshes/hx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 scale=0.001 0.001 0.001
- link finger_l_link18: geometry collision mesh filename=package://motion_controller_models/models/hx5_d20/meshes/hx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 scale=0.001 0.001 0.001; visual mesh filename=package://motion_controller_models/models/hx5_d20/meshes/hx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 scale=0.001 0.001 0.001
- link finger_l_link19: geometry collision mesh filename=package://motion_controller_models/models/hx5_d20/meshes/hx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 scale=0.001 0.001 0.001; visual mesh filename=package://motion_controller_models/models/hx5_d20/meshes/hx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 scale=0.001 0.001 0.001
- link finger_l_link2: geometry collision mesh filename=package://motion_controller_models/models/hx5_d20/meshes/hx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 scale=0.001 0.001 0.001; visual mesh filename=package://motion_controller_models/models/hx5_d20/meshes/hx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 scale=0.001 0.001 0.001
- link finger_l_link20: geometry collision mesh filename=package://motion_controller_models/models/hx5_d20/meshes/hx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 scale=0.001 0.001 0.001; visual mesh filename=package://motion_controller_models/models/hx5_d20/meshes/hx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 scale=0.001 0.001 0.001
- link finger_l_link3: geometry collision mesh filename=package://motion_controller_models/models/hx5_d20/meshes/hx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 scale=0.001 0.001 0.001; visual mesh filename=package://motion_controller_models/models/hx5_d20/meshes/hx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 scale=0.001 0.001 0.001
- link finger_l_link4: geometry collision mesh filename=package://motion_controller_models/models/hx5_d20/meshes/hx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 scale=0.001 0.001 0.001; visual mesh filename=package://motion_controller_models/models/hx5_d20/meshes/hx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 scale=0.001 0.001 0.001
- link finger_l_link5: geometry collision mesh filename=package://motion_controller_models/models/hx5_d20/meshes/hx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 scale=0.001 0.001 0.001; visual mesh filename=package://motion_controller_models/models/hx5_d20/meshes/hx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 scale=0.001 0.001 0.001
- link finger_l_link6: geometry collision mesh filename=package://motion_controller_models/models/hx5_d20/meshes/hx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 scale=0.001 0.001 0.001; visual mesh filename=package://motion_controller_models/models/hx5_d20/meshes/hx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 scale=0.001 0.001 0.001
- link finger_l_link7: geometry collision mesh filename=package://motion_controller_models/models/hx5_d20/meshes/hx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 scale=0.001 0.001 0.001; visual mesh filename=package://motion_controller_models/models/hx5_d20/meshes/hx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 scale=0.001 0.001 0.001
- link finger_l_link8: geometry collision mesh filename=package://motion_controller_models/models/hx5_d20/meshes/hx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 scale=0.001 0.001 0.001; visual mesh filename=package://motion_controller_models/models/hx5_d20/meshes/hx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 scale=0.001 0.001 0.001
- link finger_l_link9: geometry collision mesh filename=package://motion_controller_models/models/hx5_d20/meshes/hx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 scale=0.001 0.001 0.001; visual mesh filename=package://motion_controller_models/models/hx5_d20/meshes/hx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 scale=0.001 0.001 0.001
- link hx5_d20_left_base: geometry collision mesh filename=package://motion_controller_models/models/hx5_d20/meshes/hx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 scale=0.001 0.001 0.001; visual mesh filename=package://motion_controller_models/models/hx5_d20/meshes/hx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 scale=0.001 0.001 0.001

File: motion_controller_models/models/hx5_d20/hx5_d20_right.urdf (robot description, URDF)
Before this commit: robot hx5_d20_right, 26 links, 25 joints
Links:
- link finger_end_r_link1: geometry visual box size=0.01 0.01 0.01
- link finger_end_r_link2: geometry visual box size=0.01 0.01 0.01
- link finger_end_r_link3: geometry visual box size=0.01 0.01 0.01
- link finger_end_r_link4: geometry visual box size=0.01 0.01 0.01
- link finger_end_r_link5: geometry visual box size=0.01 0.01 0.01
- link finger_r_link1: geometry collision mesh filename=package://ffw_description/meshes/common/hx5_d20/hx5_d20_rig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 scale=0.001 0.001 0.001; visual mesh filename=package://ffw_description/meshes/common/hx5_d20/hx5_d20_rig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 scale=0.001 0.001 0.001
- link finger_r_link10: geometry collision mesh filename=package://ffw_description/meshes/common/hx5_d20/hx5_d20_rig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 scale=0.001 0.001 0.001; visual mesh filename=package://ffw_description/meshes/common/hx5_d20/hx5_d20_rig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 scale=0.001 0.001 0.001
- link finger_r_link11: geometry collision mesh filename=package://ffw_description/meshes/common/hx5_d20/hx5_d20_rig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 scale=0.001 0.001 0.001; visual mesh filename=package://ffw_description/meshes/common/hx5_d20/hx5_d20_rig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 scale=0.001 0.001 0.001
- link finger_r_link12: geometry collision mesh filename=package://ffw_description/meshes/common/hx5_d20/hx5_d20_rig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 scale=0.001 0.001 0.001; visual mesh filename=package://ffw_description/meshes/common/hx5_d20/hx5_d20_rig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 scale=0.001 0.001 0.001
- link finger_r_link13: geometry collision mesh filename=package://ffw_description/meshes/common/hx5_d20/hx5_d20_rig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 scale=0.001 0.001 0.001; visual mesh filename=package://ffw_description/meshes/common/hx5_d20/hx5_d20_rig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 scale=0.001 0.001 0.001
- link finger_r_link14: geometry collision mesh filename=package://ffw_description/meshes/common/hx5_d20/hx5_d20_rig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 scale=0.001 0.001 0.001; visual mesh filename=package://ffw_description/meshes/common/hx5_d20/hx5_d20_rig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 scale=0.001 0.001 0.001
- link finger_r_link15: geometry collision mesh filename=package://ffw_description/meshes/common/hx5_d20/hx5_d20_rig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 scale=0.001 0.001 0.001; visual mesh filename=package://ffw_description/meshes/common/hx5_d20/hx5_d20_rig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 scale=0.001 0.001 0.001
- link finger_r_link16: geometry collision mesh filename=package://ffw_description/meshes/common/hx5_d20/hx5_d20_rig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 scale=0.001 0.001 0.001; visual mesh filename=package://ffw_description/meshes/common/hx5_d20/hx5_d20_rig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 scale=0.001 0.001 0.001
- link finger_r_link17: geometry collision mesh filename=package://ffw_description/meshes/common/hx5_d20/hx5_d20_rig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 scale=0.001 0.001 0.001; visual mesh filename=package://ffw_description/meshes/common/hx5_d20/hx5_d20_rig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 scale=0.001 0.001 0.001
- link finger_r_link18: geometry collision mesh filename=package://ffw_description/meshes/common/hx5_d20/hx5_d20_rig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 scale=0.001 0.001 0.001; visual mesh filename=package://ffw_description/meshes/common/hx5_d20/hx5_d20_rig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 scale=0.001 0.001 0.001
- link finger_r_link19: geometry collision mesh filename=package://ffw_description/meshes/common/hx5_d20/hx5_d20_rig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 scale=0.001 0.001 0.001; visual mesh filename=package://ffw_description/meshes/common/hx5_d20/hx5_d20_rig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 scale=0.001 0.001 0.001
- link finger_r_link2: geometry collision mesh filename=package://ffw_description/meshes/common/hx5_d20/hx5_d20_rig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 scale=0.001 0.001 0.001; visual mesh filename=package://ffw_description/meshes/common/hx5_d20/hx5_d20_rig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 scale=0.001 0.001 0.001
- link finger_r_link20: geometry collision mesh filename=package://ffw_description/meshes/common/hx5_d20/hx5_d20_rig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 scale=0.001 0.001 0.001; visual mesh filename=package://ffw_description/meshes/common/hx5_d20/hx5_d20_rig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 scale=0.001 0.001 0.001
- link finger_r_link3: geometry collision mesh filename=package://ffw_description/meshes/common/hx5_d20/hx5_d20_rig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 scale=0.001 0.001 0.001; visual mesh filename=package://ffw_description/meshes/common/hx5_d20/hx5_d20_rig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 scale=0.001 0.001 0.001
- link finger_r_link4: geometry collision mesh filename=package://ffw_description/meshes/common/hx5_d20/hx5_d20_rig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 scale=0.001 0.001 0.001; visual mesh filename=package://ffw_description/meshes/common/hx5_d20/hx5_d20_rig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 scale=0.001 0.001 0.001
- link finger_r_link5: geometry collision mesh filename=package://ffw_description/meshes/common/hx5_d20/hx5_d20_rig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 scale=0.001 0.001 0.001; visual mesh filename=package://ffw_description/meshes/common/hx5_d20/hx5_d20_rig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 scale=0.001 0.001 0.001
- link finger_r_link6: geometry collision mesh filename=package://ffw_description/meshes/common/hx5_d20/hx5_d20_rig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 scale=0.001 0.001 0.001; visual mesh filename=package://ffw_description/meshes/common/hx5_d20/hx5_d20_rig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 scale=0.001 0.001 0.001
- link finger_r_link7: geometry collision mesh filename=package://ffw_description/meshes/common/hx5_d20/hx5_d20_rig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 scale=0.001 0.001 0.001; visual mesh filename=package://ffw_description/meshes/common/hx5_d20/hx5_d20_rig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 scale=0.001 0.001 0.001
- link finger_r_link8: geometry collision mesh filename=package://ffw_description/meshes/common/hx5_d20/hx5_d20_rig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 scale=0.001 0.001 0.001; visual mesh filename=package://ffw_description/meshes/common/hx5_d20/hx5_d20_rig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 scale=0.001 0.001 0.001
- link finger_r_link9: geometry collision mesh filename=package://ffw_description/meshes/common/hx5_d20/hx5_d20_rig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 scale=0.001 0.001 0.001; visual mesh filename=package://ffw_description/meshes/common/hx5_d20/hx5_d20_rig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 scale=0.001 0.001 0.001
- link hx5_d20_right_base: geometry collision mesh filename=package://ffw_description/meshes/common/hx5_d20/hx5_d20_rig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 scale=0.001 0.001 0.001; visual mesh filename=package://ffw_description/meshes/common/hx5_d20/hx5_d20_rig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 scale=0.001 0.001 0.001
