Commit message: Fixed error

File: motion_controller_models/models/omy/omy_f3m.urdf (robot description, URDF)
Before this commit: robot omy_f3m, 15 links, 14 joints
Links:
- link rh_p12_rn_base: geometry visual mesh filename=package://open_manipulator_description/meshes/rh_p12_rn_a/b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 scale=0.001 0.001 0.001
- link rh_p12_rn_l1: geometry visual mesh filename=package://open_manipulator_description/meshes/rh_p12_rn_a/l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 scale=0.001 0.001 0.001
- link rh_p12_rn_l2: geometry visual mesh filename=package://open_manipulator_description/meshes/rh_p12_rn_a/l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 scale=0.001 0.001 0.001
- link rh_p12_rn_r1: geometry visual mesh filename=package://open_manipulator_description/meshes/rh_p12_rn_a/r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 scale=0.001 0.001 0.001
- link rh_p12_rn_r2: geometry visual mesh filename=package://open_manipulator_description/meshes/rh_p12_rn_a/r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 scale=0.001 0.001 0.001
